Commit message: Update seekurjr.urdf.xacro

File: urdf/seekurjr.urdf.xacro (robot description, xacro)
@@ -34,5 +34,5 @@
 	  </visual>
 	</link>
-  <link name="laser">
+  <link name="base_laser">
     <visual>
       <geometry name="skj_laser">
@@ -47,5 +47,5 @@
     <origin xyz="0.51 0 0.3" rpy="0 0 0"/>
     <parent link="base_link"/>
-    <child link="laser"/>
+    <child link="base_laser"/>
   </joint>
   <xacro:macro name="skj_wheel" params="end side endreflect sidereflect">
